Commit message: Removendo arquivos defasados
Signed-off-by: Gabriel Alves Silva <gabriel_cte@outlook.com>

File: src/cubesat_pkg/urdf/cubesat.urdf.xacro (robot description, xacro)
@@ -5,5 +5,5 @@
     <link name="world"></link>
     <joint name="1U_joint" type="floating">
-    	<origin xyz="0 0 0" rpy="0 0 0"/>
+    	<origin xyz="0 0 0.5" rpy="0 0 0"/>
     	<parent link="world"/>
     	<child link="1U_link"/>
